File: LV8548MC/PCB/LV8548MC.kicad_pcb (KiCad board)
At the start: 2 copper layers, 10 parts, among them J1 Conn_01x08_Socket, J2 Conn_01x02_Pin, J3 Conn_01x08_Pin, U1 LV8548MC, U2 LV8548MC, U4 L7805

Commit message: LV8548MC基板
Parts:
- U4: footprint Package_TO_SOT_THT:TO-220-3_Horizontal_TabUp -> Package_TO_SOT_THT:TO-220-3_Horizontal_TabDown
- moved J3 18.0 mm to (152.4, 104.1)
- moved U4 5.08 mm to (127.0, 121.9), turned to 0 degrees
- moved C3 2.94 mm to (146.8, 119.9)
- moved U2 2.94 mm to (146.8, 116.1)
- moved C4 2.94 mm to (146.8, 112.3)
- moved U1 2.94 mm to (146.8, 108.5)
- moved C2 2.64 mm to (130.8, 120.4), turned to 180 degrees
- moved C1 2.63 mm to (128.3, 123.4), turned to 0 degrees
Connections:
- J1 pad 1: unconnected-(J1-Pin_1-Pad1) -> Net-(J1-Pin_1)
- J1 pad 2: unconnected-(J1-Pin_2-Pad2) -> Net-(J1-Pin_2)
- J1 pad 3: unconnected-(J1-Pin_3-Pad3) -> Net-(J1-Pin_3)
- J1 pad 4: unconnected-(J1-Pin_4-Pad4) -> Net-(J1-Pin_4)
- J1 pad 5: unconnected-(J1-Pin_5-Pad5) -> Net-(J1-Pin_5)
- J1 pad 6: unconnected-(J1-Pin_6-Pad6) -> Net-(J1-Pin_6)
- J1 pad 7: unconnected-(J1-Pin_7-Pad7) -> Net-(J1-Pin_7)
- J1 pad 8: unconnected-(J1-Pin_8-Pad8) -> Net-(J1-Pin_8)
- J3 pad 1: unconnected-(J3-Pin_1-Pad1) -> Net-(J3-Pin_1)
- J3 pad 2: unconnected-(J3-Pin_2-Pad2) -> Net-(J3-Pin_2)
- J3 pad 3: unconnected-(J3-Pin_3-Pad3) -> Net-(J3-Pin_3)
- J3 pad 4: unconnected-(J3-Pin_4-Pad4) -> Net-(J3-Pin_4)
- J3 pad 5: unconnected-(J3-Pin_5-Pad5) -> Net-(J3-Pin_5)
- J3 pad 6: unconnected-(J3-Pin_6-Pad6) -> Net-(J3-Pin_6)
- J3 pad 7: unconnected-(J3-Pin_7-Pad7) -> Net-(J3-Pin_7)
- J3 pad 8: unconnected-(J3-Pin_8-Pad8) -> Net-(J3-Pin_8)
- U1 pad 10: unconnected-(U1-OUT1-Pad10) -> Net-(J3-Pin_4)
- U1 pad 2: unconnected-(U1-IN1-Pad2) -> Net-(J1-Pin_4)
- U1 pad 3: unconnected-(U1-IN2-Pad3) -> Net-(J1-Pin_3)
- U1 pad 4: unconnected-(U1-IN3-Pad4) -> Net-(J1-Pin_2)
- U1 pad 5: unconnected-(U1-IN4-Pad5) -> Net-(J1-Pin_1)
- U1 pad 7: unconnected-(U1-OUT4-Pad7) -> Net-(J3-Pin_1)
- U1 pad 8: unconnected-(U1-OUT3-Pad8) -> Net-(J3-Pin_2)
- U1 pad 9: unconnected-(U1-OUT2-Pad9) -> Net-(J3-Pin_3)
- U2 pad 10: unconnected-(U2-OUT1-Pad10) -> Net-(J3-Pin_8)
- U2 pad 2: unconnected-(U2-IN1-Pad2) -> Net-(J1-Pin_8)
- U2 pad 3: unconnected-(U2-IN2-Pad3) -> Net-(J1-Pin_7)
- U2 pad 4: unconnected-(U2-IN3-Pad4) -> Net-(J1-Pin_6)
- U2 pad 5: unconnected-(U2-IN4-Pad5) -> Net-(J1-Pin_5)
- U2 pad 7: unconnected-(U2-OUT4-Pad7) -> Net-(J3-Pin_5)
- U2 pad 8: unconnected-(U2-OUT3-Pad8) -> Net-(J3-Pin_6)
- U2 pad 9: unconnected-(U2-OUT2-Pad9) -> Net-(J3-Pin_7)
Routing:
- net +5V: track 17.4 -> 57.5 mm
- net GND: track 17.7 -> 44.8 mm
- net Net-(J1-Pin_8): track 0.00 -> 22.5 mm
- net Net-(J1-Pin_7): track 0.00 -> 21.5 mm
- net Net-(J1-Pin_6): track 0.00 -> 20.6 mm
- net Net-(J1-Pin_5): track 0.00 -> 19.2 mm
- net Net-(J1-Pin_4): track 0.00 -> 16.0 mm
- net Net-(J1-Pin_2): track 0.00 -> 15.6 mm
- net Net-(J1-Pin_3): track 0.00 -> 15.1 mm
- net Net-(J1-Pin_1): track 0.00 -> 13.7 mm
- net +12V: track 0.00 -> 11.5 mm
- net Net-(J3-Pin_8): track 0.00 -> 5.07 mm
- net Net-(J3-Pin_1): track 0.00 -> 5.05 mm
- net Net-(J3-Pin_7): track 0.00 -> 4.14 mm
- net Net-(J3-Pin_2): track 0.00 -> 3.68 mm
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- added copper zone on B.Cu, net GND
Other:
- board outline added: 33 x 42.4 mm
