File: SerialParallelPWM/PCB/SerialParallelPWM.kicad_pcb (KiCad board)
At the start: 2 copper layers, 10 parts, among them J1 Conn_01x03_Socket, J2 Conn_01x02_Pin, J3 Conn_01x08_Pin, J4 Conn_01x02_Socket, U1 ATtiny44-20P, U2 L7805

Commit message: パラレル変換基板
Parts:
- moved U1 12.8 mm to (149.9, 111.5), turned to 180 degrees
- moved C3 9.18 mm to (146.1, 111.5), turned to 180 degrees
- moved R1 5.30 mm to (146.1, 107.7), turned to -90 degrees
Routing:
- net +5V: track 10.1 -> 44.7 mm
- net /RESET: track 11.0 -> 28.2 mm
- net /TX: track 1.27 -> 15.9 mm
- net GND: track 13.5 -> 26.8 mm
- net /P7: track 29.3 -> 18.4 mm
- net /RX: track 1.27 -> 12.2 mm
- net /P6: track 24.7 -> 14.8 mm
- net /P0: track 1.27 -> 10.7 mm
- net /P5: track 10.4 -> 3.55 mm
- net /P1: track 1.27 -> 7.15 mm
- net /P4: track 11.0 -> 7.15 mm
- net /P2: track 1.27 -> 3.55 mm
- net /P3: track 12.1 -> 10.7 mm
- net +12V: track 12.2 -> 11.4 mm
- added copper zone on B.Cu, net GND
Other:
- board outline added: 40.4 x 42.4 mm
