File: SerialParallelPWM/PCB/SerialParallelPWM.kicad_sch (KiCad schematic)
At the start: 10 parts, among them J1 Conn_01x03_Socket, J2 Conn_01x02_Pin, J3 Conn_01x08_Pin, J4 Conn_01x02_Socket, U1 ATtiny44-20P, U2 L7805

Commit message: パラレル変換基板
Other:
- moved on the sheet: C1, C2, C3, J1, J2, J3, J4, R1, U1, U2
